File: main.sch (EAGLE design)
At the start: 7 parts

Commit message: v1.1.0
Parts:
- removed JP2: (no value), MIA_LIBRARY-2-2-2:PINHD-4_DATA
- added IMU: IMU_ROBOCON_GY521, MIA_LIBRARY-2-2-2:IMU_ROBOCON_GY521
Connections:
- net 3.3V@1: now also IMU.VCC; no longer JP2.1
- net GND@1: now also IMU.GND; no longer JP2.2
- net PB_6: now also IMU.SCL; no longer JP2.3
- net PB_7: now also IMU.SDA; no longer JP2.4
Other:
- moved on the sheet: ENCODER, TTL1, TTL3, VIN
