File: main.brd (EAGLE design)
At the start: 67 x 55.5 mm, 7 parts

Commit message: v1.1.0
Parts:
- removed JP2: (no value), MIA_LIBRARY-2-2-2:1X04_DATA
- added IMU: IMU_ROBOCON_GY521, MIA_LIBRARY-2-2-2:IMU_GY521
- moved CYTRON 9.25 mm to (57.1, 54.6)
- moved ENCODER 9.25 mm to (35.6, 54.6)
- moved TTL1 9.25 mm to (31.7, 19.4)
- moved TTL3 9.25 mm to (15.2, 54.6)
- moved VIN 9.25 mm to (12.7, 19.1)
- moved U$1 9.25 mm to (34.3, 36.8)
Connections:
- net 3.3V@1: now also IMU.VCC; no longer JP2.1
- net GND@1: now also IMU.GND; no longer JP2.2
- net PB_6: now also IMU.SCL; no longer JP2.3
- net PB_7: now also IMU.SDA; no longer JP2.4
Routing:
- net 3.3V@1: track 29.3 -> 9.42 mm
- net PB_6: track 18.4 -> 30.6 mm
- net GND@1: track 76.3 -> 66.8 mm
- net PB_7: track 18.4 -> 11.5 mm
Other:
- board size 67 x 55.5 mm -> 70.8 x 64.4 mm

Commit message: v1.2.0
Routing:
- net GND@2: track 112.2 -> 121.9 mm
- net GND@1: track 66.8 -> 75.4 mm
- net 5V: track 137.4 -> 145.7 mm
- net PA_1: track 28.7 -> 31.2 mm
- net PB_6: track 30.6 -> 32.4 mm
